Commit message: Various modifications to test task

File: files/test-model.urdf (robot description, URDF)
Before this commit: robot test-robot, 6 links, 5 joints
Links:
- added link link4; collision box size=0.1 0.1 0.3; visual box size=0.1 0.1 0.3
- link effector: geometry collision sphere radius=0.071; visual sphere radius=0.071
Joints:
- added joint joint4: type revolute, parent link3, child link4, origin xyz=0 0 0.25, limit lower=-1.57 upper=1.57 effort=0 velocity=0
- joint eff_joint: parent link3 -> link4

Commit message: Minor changes to task files

File: files/test-model.urdf (robot description, URDF)
Before this commit: robot test-robot, 7 links, 6 joints
Links:
- removed link link4
- link link3: geometry collision box size=0.1 0.1 0.6; visual box size=0.1 0.1 0.6
Joints:
- removed joint joint4
- joint eff_joint: origin xyz=0 0 .25 -> xyz=0 0 .6; parent link4 -> link3
- joint joint2: limit lower=-1.57 upper=1.57 effort=0 velocity=0 -> lower=-0.1 upper=3.14 effort=0 velocity=0
- joint joint3: limit lower=-1.57 upper=1.57 effort=0 velocity=0 -> lower=-0.1 upper=3.14 effort=0 velocity=0

Commit message: Base joint is now continuous (no limits)

File: files/test-model.urdf (robot description, URDF)
Before this commit: robot test-robot, 6 links, 5 joints
Joints:
- joint world_joint: limit lower=-3.14 upper=3.14 effort=0 velocity=0 -> (none); type revolute -> continuous

Commit message: Moved effector CoM a bit further

File: files/test-model.urdf (robot description, URDF)
Before this commit: robot test-robot, 6 links, 5 joints
Joints:
- joint eff_joint: origin xyz=0 0 .6 -> xyz=0 0 .65

Commit message: Made robot pure kinematic (hopefully)

File: files/test-model.urdf (robot description, URDF)
Before this commit: robot test-robot, 6 links, 5 joints
Links:
- link effector: mass None -> 0.0
- link link0: mass None -> 0.0
- link link1: mass None -> 0.0
- link link2: mass None -> 0.0
- link link3: mass None -> 0.0

Commit message: Added limits to base joint so that PRM does not roll over

File: files/test-model.urdf (robot description, URDF)
Before this commit: robot test-robot, 6 links, 5 joints
Joints:
- joint world_joint: limit (none) -> lower=-3.14 upper=3.14 effort=0 velocity=0; type continuous -> revolute

Commit message: changed sizes of robot links

File: files/test-model.urdf (robot description, URDF)
Before this commit: robot test-robot, 6 links, 5 joints
Links:
- link link1: geometry collision box size=0.1 0.1 1.5; visual box size=0.1 0.1 1.0
- link link2: geometry collision box size=0.1 0.1 0.75; visual box size=0.1 0.1 1.0
- link link3: geometry collision box size=0.1 0.1 0.6; visual box size=0.1 0.1 1.0
Joints:
- joint eff_joint: origin xyz=0 0 .65 -> xyz=0 0 1.05
- joint joint2: origin xyz=0 0 1 -> xyz=0 0 1.0
- joint joint3: origin xyz=0 0 0.75 -> xyz=0 0 1

Commit message: Collision fixes

File: files/test-model.urdf (robot description, URDF)
Before this commit: robot test-robot, 6 links, 5 joints
Links:
- link link1: geometry collision box size=0.1 0.1 1.0; visual box size=0.1 0.1 1.0
- link link2: geometry collision box size=0.1 0.1 1.0; visual box size=0.1 0.1 1.0
- link link3: geometry collision box size=0.1 0.1 1.0; visual box size=0.1 0.1 1.0
Joints:
- joint world_joint: limit lower=-3.14 upper=3.14 effort=0 velocity=0 -> (none); type revolute -> continuous
